File: 555_Timer_Clock.kicad_pcb (KiCad board)
At the start: 2 copper layers, 39 x 25 mm, 13 parts, among them J2 CLK_Out, U1 ICM7555xB

Commit message: Update
Parts:
- added G***: LOGO, my_footprints:lumi, F.Cu at (105.5, 63.5)
- added J1: +5V, my_footprints:Terminal_Block_5mm, F.Cu at (101.5, 73.0)
- added SW1: Trigger, my_footprints:slide_switch_2.54mm, F.Cu at (123.0, 81.0)
- added SW2: RST, my_footprints:tact_switch_5mm, F.Cu at (112.5, 81.0)
Routing:
- net GND: track 0.00 -> 77.0 mm, vias 0 -> 2
- net /+5V: track 0.00 -> 37.9 mm
- net /Trigger: track 0.00 -> 35.0 mm
- net /CLK_Out: track 0.00 -> 24.7 mm, vias 0 -> 1
- net /RST: track 0.00 -> 18.1 mm
- net Net-(U1-DISCH): track 0.00 -> 12.9 mm
- net Net-(D1-K): track 0.00 -> 9.21 mm
- net Net-(U1-CONT): track 0.00 -> 7.46 mm
Other:
- board text added: "VIGILAR"

Commit message: Update
Parts:
- removed the G*** at (105.5, 63.5)
- added G***: LOGO, my_footprints:geo, F.Cu at (105.5, 63.5)
